File: Schematics/shematics angle cal/shematics angle cal.kicad_sch (KiCad schematic)
At the start: 4 parts

Commit message: Updated project files
Connections:
- new net: 0.91OLED1. (GND), AS5600. (GP0), BT1.2 (-), XIAO2. (D7)
- new net: 0.91OLED1. (GND), AS5600. (GP0), XIAO2. (D7) (x3)
- now unconnected: AS5600. (GP0), AS5600. (GP0), AS5600. (GP0), AS5600. (GP0), XIAO2. (D7), XIAO2. (D7), XIAO2. (D7), XIAO2. (D7)
Changed lines of the file:
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@@
 		(color 255 16 0 1)
 	)
+	(junction
+		(at 43.18 80.01)
+		(diameter 0)
+		(color 255 0 23 1)
+	)
 	(wire
 		(pts
@@
 	(wire
 		(pts
-			(xy 38.1 80.01) (xy 63.5 80.01)
+			(xy 38.1 80.01) (xy 43.18 80.01)
 		)
 		(stroke
@@
 	(wire
 		(pts
+			(xy 72.39 48.26) (xy 72.39 55.88)
+		)
+		(stroke
+			(width 0)
+			(type default)
+			(color 255 0 12 1)
+		)
+	)
+	(wire
+		(pts
 			(xy 78.74 71.12) (xy 111.76 71.12)
 		)
@@
 	(wire
 		(pts
+			(xy 43.18 80.01) (xy 43.18 48.26)
+		)
+		(stroke
+			(width 0)
+			(type default)
+			(color 255 0 12 1)
+		)
+	)
+	(wire
+		(pts
 			(xy 85.09 59.69) (xy 82.55 59.69)
 		)
@@
 	(wire
 		(pts
+			(xy 43.18 80.01) (xy 63.5 80.01)
+		)
+		(stroke
+			(width 0)
+			(type default)
+			(color 255 0 12 1)
+		)
+	)
+	(wire
+		(pts
 			(xy 82.55 76.2) (xy 82.55 91.44)
 		)
@@
 			(width 0)
 			(type default)
+		)
+	)
+	(wire
+		(pts
+			(xy 43.18 48.26) (xy 72.39 48.26)
+		)
+		(stroke
+			(width 0)
+			(type default)
+			(color 255 0 12 1)
 		)
 	)
@@
 		(in_pos_files yes)
 		(dnp no)
-		(fields_autoplaced yes)
 		(property "Reference" "0.91OLED1"
-			(at 113.03 90.1699 0)
-			(show_name no)
-			(do_not_autoplace no)
+			(at 100.076 89.916 0)
+			(show_name no)
+			(do_not_autoplace no)
